Commit message: 20250927

File: urdf/cooperative_transportation_4ws.xacro (robot description, xacro)
@@ -8,38 +8,43 @@
 <xacro:property name="vehicle2_Yaw" value="${-PI/8}" />
 <xacro:property name="vehicle3_Yaw" value="${PI/6}" />
+<!--各リンクの質量と慣性をfusionから変換 -->
+<!-- 荷台 -->
+<xacro:property name="fusion_carrier_mass" value="2052.2363345901408" />
+<xacro:property name="sim_carrier_mass" value="100" />
+<xacro:property name="carrier_inertia_coef" value="${sim_carrier_mass/fusion_carrier_mass}" />
+<!-- -->
+<xacro:property name="fusion_vehicle_body_mass" value="2113.272311120373" />
+<xacro:property name="sim_body_mass" value="100" />
+<xacro:property name="vehicle_inertia_coef" value="${sim_body_mass/fusion_vehicle_body_mass}" />
+<!-- 車輪 -->
+<xacro:property name="fusion_wheel_mass" value="${sim_wheel_mass}" />
+<xacro:property name="sim_wheel_mass" value="8.0" />
+<xacro:property name="wheel_inertia_coef" value="${sim_wheel_mass/fusion_wheel_mass}" />
 <xacro:property name="wheel_joint_damping" value="0.1" />
 <xacro:property name="wheel_joint_mu" value="0.001" />
 <xacro:property name="wheel_joint_friction" value="${wheel_joint_mu * 0.0}" /> <!-- 横方向に垂直抗力は生まれないため0.0 -->
-<!--各リンクの質量と慣性をfusionから変換 -->
-<xacro:property name="fusion_carrier_mass" value="2052.2363345901408" />
-<xacro:property name="sim_carrier_mass" value="100" />
-<xacro:property name="carrier_inertia_coef" value="${sim_carrier_mass/fusion_carrier_mass}" />
-<xacro:property name="fusion_vehicle_body_mass" value="2113.272311120373" />
-<xacro:property name="sim_body_mass" value="100" />
-<xacro:property name="vehicle_inertia_coef" value="${sim_body_mass/fusion_vehicle_body_mass}" />
-<!-- 荷台と連結点のmass -->
 <xacro:property name="carrier_mass" value="2052.2363345901408" />
 <xacro:property name="linkage_point_mass" value="16.301253040579397" />
 <xacro:property name="vehicle_body_mass" value="2113.272311120373" />
 <xacro:property name="sliding_mechanism_mass" value="36.58325703660448" />
-<!-- friction and damping of sliding mechanism -->
-<xacro:property name="sliding_mechanism_damping" value="${0.5*2*sqrt(100000*(carrier_mass/3 + linkage_point_mass))}" /> <!-- ばね定数：1000~10000, 割合：50%-->
-<xacro:property name="sliding_mechanism_mu" value="0.003" />
-<xacro:property name="sliding_mechanism_friction" value="${sliding_mechanism_mu*gravitational_acceleration*(carrier_mass/3 + linkage_point_mass)}" />
-<!-- friction and damping of steering -->
+<!-- 摺動機構 -->
+<xacro:property name="sliding_mechanism_damping" value="${(0.5*2*sqrt(100000*(carrier_inertia_coef/3 + linkage_point_mass)))/5.0}" /> <!-- ばね定数：1000~10000, 割合：50%-->
+<xacro:property name="sliding_mechanism_mu" value="0.3" />
+<xacro:property name="sliding_mechanism_friction" value="${sliding_mechanism_mu*gravitational_acceleration*(carrier_inertia_coef/3 + linkage_point_mass)}" />
+<!-- ステアリング -->
 <xacro:property name="steering_damping" value="5.0" />
-<xacro:property name="steering_mu" value="0.001" />
-<xacro:property name="steering_friction" value="${steering_mu * gravitational_acceleration * 0.25*(carrier_mass/3 + linkage_point_mass + sliding_mechanism_mass + vehicle_body_mass)}" />
-<!-- friction and damping of rotational joint -->
-<xacro:property name="rotational_joint_damping" value="0.1" />
+<xacro:property name="steering_mu" value="0.01" />
+<xacro:property name="steering_friction" value="${steering_mu * gravitational_acceleration * 0.25*(carrier_inertia_coef/3 + linkage_point_mass + sliding_mechanism_mass + sim_body_mass)}" />
+<!-- 摺動機構に乗っかている回転関節 -->
+<xacro:property name="rotational_joint_damping" value="0.02" />
 <xacro:property name="rotational_joint_mu" value="0.001" />
-<xacro:property name="rotational_joint_friction" value="${rotational_joint_mu * gravitational_acceleration * carrier_mass/3}" />
+<xacro:property name="rotational_joint_friction" value="${rotational_joint_mu * gravitational_acceleration * carrier_inertia_coef/3}" />
 <!-- wheelの接地面の摩擦などを定義 -->
-<xacro:property name="wheel_surface_mu1" value="0.8"/>
-<xacro:property name="wheel_surface_mu2" value="0.6" />
-<xacro:property name="wheel_kp" value="5e4" />
-<xacro:property name="wheel_kd" value="1.0" />
+<xacro:property name="wheel_surface_mu1" value="0.4"/>
+<xacro:property name="wheel_surface_mu2" value="1.0" />
+<xacro:property name="wheel_kp" value="2e4" />
+<xacro:property name="wheel_kd" value="5.0" />
 <xacro:property name="wheel_minDepth" value="0.01" />
-<xacro:property name="wheel_maxVel" value="1.0" />
+<xacro:property name="wheel_maxVel" value="0.5" />
 <xacro:include filename="$(find cooperative_transportation_4ws_description)/urdf/materials.xacro" />
 <xacro:include filename="$(find cooperative_transportation_4ws_description)/urdf/cooperative_transportation_4ws.trans" />
@@ -89,6 +94,6 @@
   <inertial>
     <origin xyz="1.7798855900252875e-07 2.54069273286639e-07 -3.1158354278637557e-07" rpy="0 0 0"/>
-    <mass value="20.149174540012407"/>
-    <inertia ixx="0.113544" iyy="0.222011" izz="0.113544" ixy="0.0" iyz="0.0" ixz="-0.0"/>
+    <mass value="${sim_wheel_mass}"/>
+    <inertia ixx="${wheel_inertia_coef*0.113544}" iyy="${wheel_inertia_coef*0.222011}" izz="${wheel_inertia_coef*0.113544}" ixy="0.0" iyz="0.0" ixz="0.0"/>
   </inertial>
   <visual>
@@ -210,5 +215,5 @@
     <origin xyz="2.5142643989006785e-07 2.5406923826604144e-07 -0.014912246259013051" rpy="0 0 0"/>
     <mass value="12.646385127140846"/>
-    <inertia ixx="0.752015" iyy="0.005192" izz="0.755318" ixy="0.0" iyz="0.0" ixz="-0.0"/>
+    <inertia ixx="0.752015" iyy="0.005192" izz="0.755318" ixy="0.0" iyz="0.0" ixz="0.0"/>
   </inertial>
   <visual>
@@ -249,6 +254,6 @@
   <inertial>
     <origin xyz="1.779885572261719e-07 2.540692008445866e-07 -3.1158354346638717e-07" rpy="0 0 0"/>
-    <mass value="20.149174540012407"/>
-    <inertia ixx="0.113544" iyy="0.222011" izz="0.113544" ixy="0.0" iyz="0.0" ixz="-0.0"/>
+    <mass value="${sim_wheel_mass}"/>
+    <inertia ixx="${wheel_inertia_coef*0.113544}" iyy="${wheel_inertia_coef*0.222011}" izz="${wheel_inertia_coef*0.113544}" ixy="0.0" iyz="0.0" ixz="0.0"/>
   </inertial>
   <visual>
@@ -269,4 +274,10 @@
           <mu>${wheel_surface_mu1}</mu>
           <mu2>${wheel_surface_mu2}</mu2>
+          <!-- fdir1: mu が作用する第1方向。ここでは「進行方向」に合わせる -->
+          <!-- タイヤ回転軸が +Y なので、進行方向はローカルX としておくのが分かりやすい -->
+          <fdir1>1 0 0</fdir1>
+          <!-- 強すぎるスティッキングを避けるためのスリップ（力依存） -->
+          <slip1>0.001</slip1>   <!-- rolling -->
+          <slip2>0.0</slip2>     <!-- lateral（基本0でOK、必要なら微小） -->
         </ode>
       </friction>
@@ -285,5 +296,5 @@
   <inertial>
     <origin xyz="1.7798855633799349e-07 2.540691992902744e-07 -3.1158354452109904e-07" rpy="0 0 0"/>
-    <mass value="20.14917454001241"/>
+    <mass value="${sim_wheel_mass}"/>
     <inertia ixx="0.113544" iyy="0.222011" izz="0.113544" ixy="-0.0" iyz="0.0" ixz="-0.0"/>
   </inertial>
@@ -305,4 +316,10 @@
           <mu>${wheel_surface_mu1}</mu>
           <mu2>${wheel_surface_mu2}</mu2>
+          <!-- fdir1: mu が作用する第1方向。ここでは「進行方向」に合わせる -->
+          <!-- タイヤ回転軸が +Y なので、進行方向はローカルX としておくのが分かりやすい -->
+          <fdir1>1 0 0</fdir1>
+          <!-- 強すぎるスティッキングを避けるためのスリップ（力依存） -->
+          <slip1>0.001</slip1>   <!-- rolling -->
+          <slip2>0.0</slip2>     <!-- lateral（基本0でOK、必要なら微小） -->
         </ode>
       </friction>
@@ -321,6 +338,6 @@
   <inertial>
     <origin xyz="1.7798855966866256e-07 2.540692710661929e-07 -3.1158354392435417e-07" rpy="0 0 0"/>
-    <mass value="20.149174540012407"/>
-    <inertia ixx="0.113544" iyy="0.222011" izz="0.113544" ixy="0.0" iyz="0.0" ixz="0.0"/>
+    <mass value="${sim_wheel_mass}"/>
+    <inertia ixx="${wheel_inertia_coef*0.113544}" iyy="${wheel_inertia_coef*0.222011}" izz="${wheel_inertia_coef*0.113544}" ixy="0.0" iyz="0.0" ixz="0.0"/>
   </inertial>
   <visual>
@@ -341,4 +358,10 @@
           <mu>${wheel_surface_mu1}</mu>
           <mu2>${wheel_surface_mu2}</mu2>
+          <!-- fdir1: mu が作用する第1方向。ここでは「進行方向」に合わせる -->
+          <!-- タイヤ回転軸が +Y なので、進行方向はローカルX としておくのが分かりやすい -->
+          <fdir1>1 0 0</fdir1>
+          <!-- 強すぎるスティッキングを避けるためのスリップ（力依存） -->
+          <slip1>0.001</slip1>   <!-- rolling -->
+          <slip2>0.0</slip2>     <!-- lateral（基本0でOK、必要なら微小） -->
         </ode>
       </friction>
@@ -358,5 +381,5 @@
     <origin xyz="2.514264050290649e-07 7.029564128707699e-08 -0.11791981845688482" rpy="0 0 0"/>
     <mass value="16.301253040579397"/>
-    <inertia ixx="0.104905" iyy="0.104905" izz="0.020865" ixy="0.0" iyz="-0.0" ixz="-0.0"/>
+    <inertia ixx="0.104905" iyy="0.104905" izz="0.020865" ixy="0.0" iyz="0.0" ixz="0.0"/>
   </inertial>
   <visual>
@@ -378,5 +401,5 @@
     <origin xyz="3.2372278280234923e-07 -1.568761989201306e-07 -0.11791981845688582" rpy="0 0 0"/>
     <mass value="16.30125304057939"/>
-    <inertia ixx="0.104905" iyy="0.104905" izz="0.020865" ixy="0.0" iyz="-0.0" ixz="-0.0"/>
+    <inertia ixx="0.104905" iyy="0.104905" izz="0.020865" ixy="0.0" iyz="0.0" ixz="0.0"/>
   </inertial>
   <visual>
@@ -438,5 +461,5 @@
     <origin xyz="3.2372281477677234e-07 2.689739853067863e-08 -0.014912246259013773" rpy="0 0 0"/>
     <mass value="12.646385127140846"/>
-    <inertia ixx="0.752015" iyy="0.005192" izz="0.755318" ixy="0.0" iyz="0.0" ixz="-0.0"/>
+    <inertia ixx="0.752015" iyy="0.005192" izz="0.755318" ixy="0.0" iyz="0.0" ixz="0.0"/>
   </inertial>
   <visual>
@@ -557,6 +580,6 @@
   <inertial>
     <origin xyz="2.5028493444434474e-07 2.689736211536342e-08 -3.1158354371618735e-07" rpy="0 0 0"/>
-    <mass value="20.149174540012407"/>
-    <inertia ixx="0.113544" iyy="0.222011" izz="0.113544" ixy="-0.0" iyz="0.0" ixz="0.0"/>
+    <mass value="${sim_wheel_mass}"/>
+    <inertia ixx="${wheel_inertia_coef*0.113544}" iyy="${wheel_inertia_coef*0.222011}" izz="${wheel_inertia_coef*0.113544}" ixy="0.0" iyz="0.0" ixz="0.0"/>
   </inertial>
   <visual>
@@ -577,4 +600,10 @@
           <mu>${wheel_surface_mu1}</mu>
           <mu2>${wheel_surface_mu2}</mu2>
+          <!-- fdir1: mu が作用する第1方向。ここでは「進行方向」に合わせる -->
+          <!-- タイヤ回転軸が +Y なので、進行方向はローカルX としておくのが分かりやすい -->
+          <fdir1>1 0 0</fdir1>
+          <!-- 強すぎるスティッキングを避けるためのスリップ（力依存） -->
+          <slip1>0.001</slip1>   <!-- rolling -->
+          <slip2>0.0</slip2>     <!-- lateral（基本0でOK、必要なら微小） -->
         </ode>
       </friction>
@@ -593,6 +622,6 @@
   <inertial>
     <origin xyz="2.5028493433332244e-07 2.6897433391681602e-08 -3.1158354339699823e-07" rpy="0 0 0"/>
-    <mass value="20.149174540012407"/>
-    <inertia ixx="0.113544" iyy="0.222011" izz="0.113544" ixy="0.0" iyz="0.0" ixz="0.0"/>
+    <mass value="${sim_wheel_mass}"/>
+    <inertia ixx="${wheel_inertia_coef*0.113544}" iyy="${wheel_inertia_coef*0.222011}" izz="${wheel_inertia_coef*0.113544}" ixy="0.0" iyz="0.0" ixz="0.0"/>
   </inertial>
   <visual>
@@ -613,4 +642,10 @@
           <mu>${wheel_surface_mu1}</mu>
           <mu2>${wheel_surface_mu2}</mu2>
+          <!-- fdir1: mu が作用する第1方向。ここでは「進行方向」に合わせる -->
+          <!-- タイヤ回転軸が +Y なので、進行方向はローカルX としておくのが分かりやすい -->
+          <fdir1>1 0 0</fdir1>
+          <!-- 強すぎるスティッキングを避けるためのスリップ（力依存） -->
+          <slip1>0.001</slip1>   <!-- rolling -->
+          <slip2>0.0</slip2>     <!-- lateral（基本0でOK、必要なら微小） -->
         </ode>
       </friction>
@@ -629,6 +664,6 @@
   <inertial>
     <origin xyz="2.5028493316758826e-07 2.6897359006738952e-08 -3.1158354495131046e-07" rpy="0 0 0"/>
-    <mass value="20.14917454001241"/>
-    <inertia ixx="0.113544" iyy="0.222011" izz="0.113544" ixy="-0.0" iyz="0.0" ixz="0.0"/>
+    <mass value="${sim_wheel_mass}"/>
+    <inertia ixx="${wheel_inertia_coef*0.113544}" iyy="${wheel_inertia_coef*0.222011}" izz="${wheel_inertia_coef*0.113544}" ixy="0.0" iyz="0.0" ixz="0.0"/>
   </inertial>
   <visual>
@@ -649,4 +684,10 @@
           <mu>${wheel_surface_mu1}</mu>
           <mu2>${wheel_surface_mu2}</mu2>
+          <!-- fdir1: mu が作用する第1方向。ここでは「進行方向」に合わせる -->
+          <!-- タイヤ回転軸が +Y なので、進行方向はローカルX としておくのが分かりやすい -->
+          <fdir1>1 0 0</fdir1>
+          <!-- 強すぎるスティッキングを避けるためのスリップ（力依存） -->
+          <slip1>0.001</slip1>   <!-- rolling -->
+          <slip2>0.0</slip2>     <!-- lateral（基本0でOK、必要なら微小） -->
         </ode>
       </friction>
@@ -665,6 +706,6 @@
   <inertial>
     <origin xyz="2.5028493477741165e-07 2.6897427618521874e-08 -3.115835443545656e-07" rpy="0 0 0"/>
-    <mass value="20.149174540012407"/>
-    <inertia ixx="0.113544" iyy="0.222011" izz="0.113544" ixy="0.0" iyz="0.0" ixz="-0.0"/>
+    <mass value="${sim_wheel_mass}"/>
+    <inertia ixx="${wheel_inertia_coef*0.113544}" iyy="${wheel_inertia_coef*0.222011}" izz="${wheel_inertia_coef*0.113544}" ixy="0.0" iyz="0.0" ixz="0.0"/>
   </inertial>
   <visual>
@@ -685,4 +726,10 @@
           <mu>${wheel_surface_mu1}</mu>
           <mu2>${wheel_surface_mu2}</mu2>
+          <!-- fdir1: mu が作用する第1方向。ここでは「進行方向」に合わせる -->
+          <!-- タイヤ回転軸が +Y なので、進行方向はローカルX としておくのが分かりやすい -->
+          <fdir1>1 0 0</fdir1>
+          <!-- 強すぎるスティッキングを避けるためのスリップ（力依存） -->
+          <slip1>0.001</slip1>   <!-- rolling -->
+          <slip2>0.0</slip2>     <!-- lateral（基本0でOK、必要なら微小） -->
         </ode>
       </friction>
@@ -722,5 +769,5 @@
     <origin xyz="1.0880185641326534e-14 7.682743330406083e-14 -0.014912246259012052" rpy="0 0 0"/>
     <mass value="12.646385127140846"/>
-    <inertia ixx="0.752015" iyy="0.005192" izz="0.755318" ixy="0.0" iyz="0.0" ixz="-0.0"/>
+    <inertia ixx="0.752015" iyy="0.005192" izz="0.755318" ixy="0.0" iyz="0.0" ixz="0.0"/>
   </inertial>
   <visual>
@@ -841,6 +888,6 @@
   <inertial>
     <origin xyz="-7.343787561397974e-08 3.930189507173054e-14 -3.1158354107940767e-07" rpy="0 0 0"/>
-    <mass value="20.149174540012407"/>
-    <inertia ixx="0.113544" iyy="0.222011" izz="0.113544" ixy="-0.0" iyz="0.0" ixz="0.0"/>
+    <mass value="${sim_wheel_mass}"/>
+    <inertia ixx="${wheel_inertia_coef*0.113544}" iyy="${wheel_inertia_coef*0.222011}" izz="${wheel_inertia_coef*0.113544}" ixy="0.0" iyz="0.0" ixz="0.0"/>
   </inertial>
   <visual>
@@ -861,4 +908,10 @@
           <mu>${wheel_surface_mu1}</mu>
           <mu2>${wheel_surface_mu2}</mu2>
+          <!-- fdir1: mu が作用する第1方向。ここでは「進行方向」に合わせる -->
+          <!-- タイヤ回転軸が +Y なので、進行方向はローカルX としておくのが分かりやすい -->
+          <fdir1>1 0 0</fdir1>
+          <!-- 強すぎるスティッキングを避けるためのスリップ（力依存） -->
+          <slip1>0.001</slip1>   <!-- rolling -->
+          <slip2>0.0</slip2>     <!-- lateral（基本0でOK、必要なら微小） -->
         </ode>
       </friction>
@@ -877,6 +930,6 @@
   <inertial>
     <origin xyz="-7.343787356006715e-08 1.1191048088221578e-13 -3.1158354157900803e-07" rpy="0 0 0"/>
-    <mass value="20.149174540012407"/>
-    <inertia ixx="0.113544" iyy="0.222011" izz="0.113544" ixy="0.0" iyz="-0.0" ixz="-0.0"/>
+    <mass value="${sim_wheel_mass}"/>
+    <inertia ixx="${wheel_inertia_coef*0.113544}" iyy="${wheel_inertia_coef*0.222011}" izz="${wheel_inertia_coef*0.113544}" ixy="0.0" iyz="0.0" ixz="0.0"/>
   </inertial>
   <visual>
@@ -897,4 +950,10 @@
           <mu>${wheel_surface_mu1}</mu>
           <mu2>${wheel_surface_mu2}</mu2>
+          <!-- fdir1: mu が作用する第1方向。ここでは「進行方向」に合わせる -->
+          <!-- タイヤ回転軸が +Y なので、進行方向はローカルX としておくのが分かりやすい -->
+          <fdir1>1 0 0</fdir1>
+          <!-- 強すぎるスティッキングを避けるためのスリップ（力依存） -->
+          <slip1>0.001</slip1>   <!-- rolling -->
+          <slip2>0.0</slip2>     <!-- lateral（基本0でOK、必要なら微小） -->
         </ode>
       </friction>
@@ -913,6 +972,6 @@
   <inertial>
     <origin xyz="-7.343787644664701e-08 3.808064974464287e-14 -3.115835421757529e-07" rpy="0 0 0"/>
-    <mass value="20.14917454001241"/>
-    <inertia ixx="0.113544" iyy="0.222011" izz="0.113544" ixy="-0.0" iyz="0.0" ixz="0.0"/>
+    <mass value="${sim_wheel_mass}"/>
+    <inertia ixx="${wheel_inertia_coef*0.113544}" iyy="${wheel_inertia_coef*0.222011}" izz="${wheel_inertia_coef*0.113544}" ixy="0.0" iyz="0.0" ixz="0.0"/>
   </inertial>
   <visual>
@@ -933,4 +992,10 @@
           <mu>${wheel_surface_mu1}</mu>
           <mu2>${wheel_surface_mu2}</mu2>
+          <!-- fdir1: mu が作用する第1方向。ここでは「進行方向」に合わせる -->
+          <!-- タイヤ回転軸が +Y なので、進行方向はローカルX としておくのが分かりやすい -->
+          <fdir1>1 0 0</fdir1>
+          <!-- 強すぎるスティッキングを避けるためのスリップ（力依存） -->
+          <slip1>0.001</slip1>   <!-- rolling -->
+          <slip2>0.0</slip2>     <!-- lateral（基本0でOK、必要なら微小） -->
         </ode>
       </friction>
@@ -949,6 +1014,6 @@
   <inertial>
     <origin xyz="-7.343787289393333e-08 1.0891287871572786e-13 -3.1158354246718645e-07" rpy="0 0 0"/>
-    <mass value="20.149174540012407"/>
-    <inertia ixx="0.113544" iyy="0.222011" izz="0.113544" ixy="0.0" iyz="0.0" ixz="0.0"/>
+    <mass value="${sim_wheel_mass}"/>
+    <inertia ixx="${wheel_inertia_coef*0.113544}" iyy="${wheel_inertia_coef*0.222011}" izz="${wheel_inertia_coef*0.113544}" ixy="0.0" iyz="0.0" ixz="0.0"/>
   </inertial>
   <visual>
@@ -969,4 +1034,10 @@
           <mu>${wheel_surface_mu1}</mu>
           <mu2>${wheel_surface_mu2}</mu2>
+          <!-- fdir1: mu が作用する第1方向。ここでは「進行方向」に合わせる -->
+          <!-- タイヤ回転軸が +Y なので、進行方向はローカルX としておくのが分かりやすい -->
+          <fdir1>1 0 0</fdir1>
+          <!-- 強すぎるスティッキングを避けるためのスリップ（力依存） -->
+          <slip1>0.001</slip1>   <!-- rolling -->
+          <slip2>0.0</slip2>     <!-- lateral（基本0でOK、必要なら微小） -->
         </ode>
       </friction>
@@ -1000,4 +1071,12 @@
       <mesh filename="package://cooperative_transportation_4ws_description/meshes/v1_sliding_machine_1.stl" scale="0.001 0.001 0.001"/>
     </geometry>
+    <surface>
+      <friction>
+        <ode>
+          <mu>${sliding_mechanism_mu}</mu>
+          <mu2>${sliding_mechanism_mu}</mu2>
+        </ode>
+      </friction>
+      </surface>
   </collision>
 </link>
@@ -1020,4 +1099,12 @@
       <mesh filename="package://cooperative_transportation_4ws_description/meshes/v2_sliding_machine_1.stl" scale="0.001 0.001 0.001"/>
     </geometry>
+    <surface>
+      <friction>
+        <ode>
+          <mu>${sliding_mechanism_mu}</mu>
+          <mu2>${sliding_mechanism_mu}</mu2>
+        </ode>
+      </friction>
+      </surface>
   </collision>
 </link>
@@ -1040,4 +1127,12 @@
       <mesh filename="package://cooperative_transportation_4ws_description/meshes/v3_sliding_machine_1.stl" scale="0.001 0.001 0.001"/>
     </geometry>
+    <surface>
+      <friction>
+        <ode>
+          <mu>${sliding_mechanism_mu}</mu>
+          <mu2>${sliding_mechanism_mu}</mu2>
+        </ode>
+      </friction>
+      </surface>
   </collision>
 </link>
@@ -1047,5 +1142,5 @@
   <child link="carrier"/>
 </joint> -->
-<joint name="carrier" type="fixed">
+<joint name="carrier_fixed" type="fixed">
   <origin xyz="0 0 0.6559999999999989" rpy="0 0 0"/>
   <parent link="base_link"/>
@@ -1058,4 +1153,5 @@
   <dynamics damping="${wheel_joint_damping}" friction="${wheel_joint_friction}"/>
   <axis xyz="0.0 1.0 -0.0"/>
+  <limit effort="40.0" velocity="200.0"/>
 </joint>
 <joint name="v1_rear_right_steering" type="revolute">
@@ -1112,4 +1208,5 @@
   <dynamics damping="${wheel_joint_damping}" friction="${wheel_joint_friction}"/>
   <axis xyz="0.0 1.0 -0.0"/>
+  <limit effort="40.0" velocity="200.0"/>
 </joint>
 <joint name="v1_front_left_wheel_rotation" type="continuous">
@@ -1119,4 +1216,5 @@
   <dynamics damping="${wheel_joint_damping}" friction="${wheel_joint_friction}"/>
   <axis xyz="0.0 1.0 -0.0"/>
+  <limit effort="40.0" velocity="200.0"/>
 </joint>
 <joint name="v1_rear_left_wheel_rotation" type="continuous">
@@ -1126,4 +1224,5 @@
   <dynamics damping="${wheel_joint_damping}" friction="${wheel_joint_friction}"/>
   <axis xyz="0.0 1.0 -0.0"/>
+  <limit effort="40.0" velocity="200.0"/>
 </joint>
 <!-- <joint name="linkage1_rotation" type="continuous">
@@ -1153,4 +1252,6 @@
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