Commit message: 20250928

File: urdf/cooperative_transportation_4ws.xacro (robot description, xacro)
@@ -1161,5 +1161,5 @@
   <dynamics damping="${steering_damping}" friction="${steering_friction}"/>
   <axis xyz="0.0 0.0 1.0"/>
-  <limit upper="1.2" lower="-1.2" effort="100" velocity="100"/>
+  <limit upper="1.57" lower="-1.57" effort="100" velocity="100"/>
 </joint>
 <joint name="v1_front_right_steering" type="revolute">
@@ -1169,5 +1169,5 @@
   <dynamics damping="${steering_damping}" friction="${steering_friction}"/>
   <axis xyz="0.0 0.0 1.0"/>
-  <limit upper="1.2" lower="-1.2" effort="100" velocity="100"/>
+  <limit upper="1.57" lower="-1.57" effort="100" velocity="100"/>
 </joint>
 <joint name="v1_front_left_steering" type="revolute">
@@ -1177,5 +1177,5 @@
   <dynamics damping="${steering_damping}" friction="${steering_friction}"/>
   <axis xyz="0.0 0.0 1.0"/>
-  <limit upper="1.2" lower="-1.2" effort="100" velocity="100"/>
+  <limit upper="1.57" lower="-1.57" effort="100" velocity="100"/>
 </joint>
 <joint name="v1_rear_left_steering" type="revolute">
@@ -1185,5 +1185,5 @@
   <dynamics damping="${steering_damping}" friction="${steering_friction}"/>
   <axis xyz="0.0 0.0 1.0"/>
-  <limit upper="1.2" lower="-1.2" effort="100" velocity="100"/>
+  <limit upper="1.57" lower="-1.57" effort="100" velocity="100"/>
 </joint>
 <joint name="v1_sliding_machine_to_body" type="fixed">
@@ -1292,5 +1292,5 @@
   <dynamics damping="${steering_damping}" friction="${steering_friction}"/>
   <axis xyz="0.0 0.0 1.0"/>
-  <limit upper="1.2" lower="-1.2" effort="100" velocity="100"/>
+  <limit upper="1.57" lower="-1.57" effort="100" velocity="100"/>
 </joint>
 <joint name="v2_rear_right_steering" type="revolute">
@@ -1300,5 +1300,5 @@
   <dynamics damping="${steering_damping}" friction="${steering_friction}"/>
   <axis xyz="0.0 0.0 1.0"/>
-  <limit upper="1.2" lower="-1.2" effort="100" velocity="100"/>
+  <limit upper="1.57" lower="-1.57" effort="100" velocity="100"/>
 </joint>
 <joint name="v2_front_left_steering" type="revolute">
@@ -1308,5 +1308,5 @@
   <dynamics damping="${steering_damping}" friction="${steering_friction}"/>
   <axis xyz="0.0 0.0 1.0"/>
-  <limit upper="1.2" lower="-1.2" effort="100" velocity="100"/>
+  <limit upper="1.57" lower="-1.57" effort="100" velocity="100"/>
 </joint>
 <joint name="v2_rear_left_steering" type="revolute">
@@ -1316,5 +1316,5 @@
   <dynamics damping="${steering_damping}" friction="${steering_friction}"/>
   <axis xyz="0.0 0.0 1.0"/>
-  <limit upper="1.2" lower="-1.2" effort="100" velocity="100"/>
+  <limit upper="1.57" lower="-1.57" effort="100" velocity="100"/>
 </joint>
 <joint name="v2_front_right_wheel_rotation" type="continuous">
@@ -1371,5 +1371,5 @@
   <dynamics damping="${steering_damping}" friction="${steering_friction}"/>
   <axis xyz="-0.0 0.0 1.0"/>
-  <limit upper="1.2" lower="-1.2" effort="100" velocity="100"/>
+  <limit upper="1.57" lower="-1.57" effort="100" velocity="100"/>
 </joint>
 <joint name="v3_rear_right_steering" type="revolute">
@@ -1379,5 +1379,5 @@
   <dynamics damping="${steering_damping}" friction="${steering_friction}"/>
   <axis xyz="-0.0 0.0 1.0"/>
-  <limit upper="1.2" lower="-1.2" effort="100" velocity="100"/>
+  <limit upper="1.57" lower="-1.57" effort="100" velocity="100"/>
 </joint>
 <joint name="v3_front_left_steering" type="revolute">
@@ -1387,5 +1387,5 @@
   <dynamics damping="${steering_damping}" friction="${steering_friction}"/>
   <axis xyz="-0.0 0.0 1.0"/>
-  <limit upper="1.2" lower="-1.2" effort="100" velocity="100"/>
+  <limit upper="1.57" lower="-1.57" effort="100" velocity="100"/>
 </joint>
 <joint name="v3_rear_left_steering" type="revolute">
@@ -1395,5 +1395,5 @@
   <dynamics damping="${steering_damping}" friction="${steering_friction}"/>
   <axis xyz="-0.0 0.0 1.0"/>
-  <limit upper="1.2" lower="-1.2" effort="100" velocity="100"/>
+  <limit upper="1.57" lower="-1.57" effort="100" velocity="100"/>
 </joint>
 <joint name="v3_front_right_wheel_rotation" type="continuous">

Commit message: 20251001

File: urdf/cooperative_transportation_4ws.xacro (robot description, xacro)
@@ -41,5 +41,5 @@
 <xacro:property name="rotational_joint_friction" value="${rotational_joint_mu * gravitational_acceleration * carrier_inertia_coef/3}" />
 <!-- wheelの接地面の摩擦などを定義 -->
-<xacro:property name="wheel_surface_mu1" value="0.4"/>
+<xacro:property name="wheel_surface_mu1" value="1.0"/>
 <xacro:property name="wheel_surface_mu2" value="1.0" />
 <xacro:property name="wheel_kp" value="2e4" />

Commit message: Change the initial position to ｙ = 1.0.

File: urdf/cooperative_transportation_4ws.xacro (robot description, xacro)
@@ -33,6 +33,6 @@
 <xacro:property name="sliding_mechanism_friction" value="${sliding_mechanism_mu*gravitational_acceleration*(carrier_inertia_coef/3 + linkage_point_mass)}" />
 <!-- ステアリング -->
-<xacro:property name="steering_damping" value="5.0" />
-<xacro:property name="steering_mu" value="0.01" />
+<xacro:property name="steering_damping" value="1.0" />
+<xacro:property name="steering_mu" value="0.001" />
 <xacro:property name="steering_friction" value="${steering_mu * gravitational_acceleration * 0.25*(carrier_inertia_coef/3 + linkage_point_mass + sliding_mechanism_mass + sim_body_mass)}" />
 <!-- 摺動機構に乗っかている回転関節 -->
@@ -1153,5 +1153,5 @@
   <dynamics damping="${wheel_joint_damping}" friction="${wheel_joint_friction}"/>
   <axis xyz="0.0 1.0 -0.0"/>
-  <limit effort="40.0" velocity="200.0"/>
+  <limit effort="100.0" velocity="200.0"/>
 </joint>
 <joint name="v1_rear_right_steering" type="revolute">
@@ -1208,5 +1208,5 @@
   <dynamics damping="${wheel_joint_damping}" friction="${wheel_joint_friction}"/>
   <axis xyz="0.0 1.0 -0.0"/>
-  <limit effort="40.0" velocity="200.0"/>
+  <limit effort="100.0" velocity="200.0"/>
 </joint>
 <joint name="v1_front_left_wheel_rotation" type="continuous">
@@ -1216,5 +1216,5 @@
   <dynamics damping="${wheel_joint_damping}" friction="${wheel_joint_friction}"/>
   <axis xyz="0.0 1.0 -0.0"/>
-  <limit effort="40.0" velocity="200.0"/>
+  <limit effort="100.0" velocity="200.0"/>
 </joint>
 <joint name="v1_rear_left_wheel_rotation" type="continuous">
@@ -1224,5 +1224,5 @@
   <dynamics damping="${wheel_joint_damping}" friction="${wheel_joint_friction}"/>
   <axis xyz="0.0 1.0 -0.0"/>
-  <limit effort="40.0" velocity="200.0"/>
+  <limit effort="100.0" velocity="200.0"/>
 </joint>
 <!-- <joint name="linkage1_rotation" type="continuous">
@@ -1324,5 +1324,5 @@
   <dynamics damping="${wheel_joint_damping}" friction="${wheel_joint_friction}"/>
   <axis xyz="0.0 1.0 -0.0"/>
-  <limit effort="40.0" velocity="200.0"/>
+  <limit effort="100.0" velocity="200.0"/>
 </joint>
 <joint name="v2_rear_right_wheel_rotation" type="continuous">
@@ -1332,5 +1332,5 @@
   <dynamics damping="${wheel_joint_damping}" friction="${wheel_joint_friction}"/>
   <axis xyz="-0.0 1.0 -0.0"/>
-  <limit effort="40.0" velocity="200.0"/>
+  <limit effort="100.0" velocity="200.0"/>
 </joint>
 <joint name="v2_front_left_wheel_rotation" type="continuous">
@@ -1340,5 +1340,5 @@
   <dynamics damping="${wheel_joint_damping}" friction="${wheel_joint_friction}"/>
   <axis xyz="0.0 1.0 -0.0"/>
-  <limit effort="40.0" velocity="200.0"/>
+  <limit effort="100.0" velocity="200.0"/>
 </joint>
 <joint name="v2_rear_left_wheel_rotation" type="continuous">
@@ -1348,5 +1348,5 @@
   <dynamics damping="${wheel_joint_damping}" friction="${wheel_joint_friction}"/>
   <axis xyz="-0.0 1.0 -0.0"/>
-  <limit effort="40.0" velocity="200.0"/>
+  <limit effort="100.0" velocity="200.0"/>
 </joint>
 <joint name="v3_sliding_machine_to_body" type="fixed">
@@ -1403,5 +1403,5 @@
   <dynamics damping="${wheel_joint_damping}" friction="${wheel_joint_friction}"/>
   <axis xyz="0.0 1.0 -0.0"/>
-  <limit effort="40.0" velocity="200.0"/>
+  <limit effort="100.0" velocity="200.0"/>
 </joint>
 <joint name="v3_rear_right_wheel_rotation" type="continuous">
@@ -1411,5 +1411,5 @@
   <dynamics damping="${wheel_joint_damping}" friction="${wheel_joint_friction}"/>
   <axis xyz="0.0 1.0 -0.0"/>
-  <limit effort="40.0" velocity="200.0"/>
+  <limit effort="100.0" velocity="200.0"/>
 </joint>
 <joint name="v3_front_left_wheel_rotation" type="continuous">
@@ -1419,5 +1419,5 @@
   <dynamics damping="${wheel_joint_damping}" friction="${wheel_joint_friction}"/>
   <axis xyz="0.0 1.0 -0.0"/>
-  <limit effort="40.0" velocity="200.0"/>
+  <limit effort="100.0" velocity="200.0"/>
 </joint>
 <joint name="v3_rear_left_wheel_rotation" type="continuous">
@@ -1427,5 +1427,5 @@
   <dynamics damping="${wheel_joint_damping}" friction="${wheel_joint_friction}"/>
   <axis xyz="0.0 1.0 -0.0"/>
-  <limit effort="40.0" velocity="200.0"/>
+  <limit effort="100.0" velocity="200.0"/>
 </joint>
 <joint name="linkage_point_to_v1" type="prismatic">

Commit message: 20251006

File: urdf/cooperative_transportation_4ws.xacro (robot description, xacro)
@@ -4,8 +4,10 @@
 <xacro:property name="gravitational_acceleration" value="9.8" />
 <xacro:property name="vehicle1_Yaw" value="0" />
+<!-- フォームクロージャー -->
 <!-- <xacro:property name="vehicle2_Yaw" value="${-PI/8}" />
 <xacro:property name="vehicle3_Yaw" value="${PI/6}" /> -->
-<xacro:property name="vehicle2_Yaw" value="${-PI/8}" />
-<xacro:property name="vehicle3_Yaw" value="${PI/6}" />
+<!-- 車両の姿勢を接線方位角に一致 -->
+<xacro:property name="vehicle2_Yaw" value="${0.0}" />
+<xacro:property name="vehicle3_Yaw" value="${0.0}" />
 <!--各リンクの質量と慣性をfusionから変換 -->
 <!-- 荷台 -->
@@ -42,5 +44,5 @@
 <!-- wheelの接地面の摩擦などを定義 -->
 <xacro:property name="wheel_surface_mu1" value="1.0"/>
-<xacro:property name="wheel_surface_mu2" value="1.0" />
+<xacro:property name="wheel_surface_mu2" value="0.8" />
 <xacro:property name="wheel_kp" value="2e4" />
 <xacro:property name="wheel_kd" value="5.0" />
@@ -78,5 +80,5 @@
   </inertial>
   <visual>
-    <origin xyz="0 0 -0.6559999999999989" rpy="0 0 0"/>
+    <origin xyz="0 -0.057 -0.6559999999999989" rpy="0 0 0"/>
     <geometry>
       <mesh filename="package://cooperative_transportation_4ws_newwheel_description/meshes/base_link.stl" scale="0.001 0.001 0.001"/>
@@ -85,5 +87,5 @@
   </visual>
   <collision>
-    <origin xyz="0 0 -0.6559999999999989" rpy="0 0 0"/>
+    <origin xyz="0 -0.057 -0.6559999999999989" rpy="0 0 0"/>
     <geometry>
       <mesh filename="package://cooperative_transportation_4ws_newwheel_description/meshes/base_link.stl" scale="0.001 0.001 0.001"/>
@@ -107,5 +109,5 @@
     <origin xyz="0 0 0" rpy="1.57 0 0"/>
     <geometry>
-      <cylinder radius="0.153" length="0.05"/>
+      <cylinder radius="0.153" length="0.07"/>
     </geometry>
   </collision>
@@ -267,5 +269,5 @@
     <origin xyz="0 0 0" rpy="1.57 0 0"/>
     <geometry>
-      <cylinder radius="0.153" length="0.05"/>
+      <cylinder radius="0.153" length="0.07"/>
     </geometry>
     <surface>
@@ -309,5 +311,5 @@
     <origin xyz="0 0 0" rpy="1.57 0 0"/>
     <geometry>
-      <cylinder radius="0.153" length="0.05"/>
+      <cylinder radius="0.153" length="0.07"/>
     </geometry>
     <surface>
@@ -351,5 +353,5 @@
     <origin xyz="0 0 0" rpy="1.57 0 0"/>
     <geometry>
-      <cylinder radius="0.153" length="0.05"/>
+      <cylinder radius="0.153" length="0.07"/>
     </geometry>
     <surface>
@@ -593,5 +595,5 @@
     <origin xyz="0 0 0" rpy="1.57 0 0"/>
     <geometry>
-      <cylinder radius="0.153" length="0.05"/>
+      <cylinder radius="0.153" length="0.07"/>
     </geometry>
     <surface>
@@ -635,5 +637,5 @@
     <origin xyz="0 0 0" rpy="1.57 0 0"/>
     <geometry>
-      <cylinder radius="0.153" length="0.05"/>
+      <cylinder radius="0.153" length="0.07"/>
     </geometry>
     <surface>
@@ -677,5 +679,5 @@
     <origin xyz="0 0 0" rpy="1.57 0 0"/>
     <geometry>
-      <cylinder radius="0.153" length="0.05"/>
+      <cylinder radius="0.153" length="0.07"/>
     </geometry>
     <surface>
@@ -719,5 +721,5 @@
     <origin xyz="0 0 0" rpy="1.57 0 0"/>
     <geometry>
-      <cylinder radius="0.153" length="0.05"/>
+      <cylinder radius="0.153" length="0.07"/>
     </geometry>
     <surface>
@@ -901,5 +903,5 @@
     <origin xyz="0 0 0" rpy="1.57 0 0"/>
     <geometry>
-      <cylinder radius="0.153" length="0.05"/>
+      <cylinder radius="0.153" length="0.07"/>
     </geometry>
     <surface>
@@ -943,5 +945,5 @@
     <origin xyz="0 0 0" rpy="1.57 0 0"/>
     <geometry>
-      <cylinder radius="0.153" length="0.05"/>
+      <cylinder radius="0.153" length="0.07"/>
     </geometry>
     <surface>
@@ -985,5 +987,5 @@
     <origin xyz="0 0 0" rpy="1.57 0 0"/>
     <geometry>
-      <cylinder radius="0.153" length="0.05"/>
+      <cylinder radius="0.153" length="0.07"/>
     </geometry>
     <surface>
@@ -1027,5 +1029,5 @@
     <origin xyz="0 0 0" rpy="1.57 0 0"/>
     <geometry>
-      <cylinder radius="0.153" length="0.05"/>
+      <cylinder radius="0.153" length="0.07"/>
     </geometry>
     <surface>
@@ -1248,24 +1250,24 @@
 </joint> -->
 <joint name="linkage1_rotation" type="continuous">
-  <origin xyz="1.60045 0.057547 0.025" rpy="0 0 ${vehicle1_Yaw}"/>
+  <origin xyz="1.60045 0.0 0.025" rpy="0 0 ${vehicle1_Yaw}"/>
   <parent link="carrier"/>
   <child link="linkage_point1_1"/>
-  <axis xyz="0.0 -0.0 -1.0"/>
+  <axis xyz="0.0 -0.0 1.0"/>
   <dynamics damping="${rotational_joint_damping}" friction="${rotational_joint_friction}"/>
   <limit effort="100" velocity="100"/>
 </joint>
 <joint name="linkage2_rotation" type="continuous">
-  <origin xyz="-0.799387 1.443222 0.025" rpy="0 0 ${vehicle2_Yaw}"/>
+  <origin xyz="-0.799387 1.386222 0.025" rpy="0 0 ${vehicle2_Yaw}"/>
   <parent link="carrier"/>
   <child link="linkage_point2_1"/>
-  <axis xyz="0.0 -0.0 -1.0"/>
+  <axis xyz="0.0 -0.0 1.0"/>
   <dynamics damping="${rotational_joint_damping}" friction="${rotational_joint_friction}"/>
   <limit effort="100" velocity="100"/>
 </joint>
 <joint name="linkage3_rotation" type="continuous">
-  <origin xyz="-0.8 -1.329973 0.025" rpy="0 0 ${vehicle3_Yaw}"/>
+  <origin xyz="-0.8 -1.386973 0.025" rpy="0 0 ${vehicle3_Yaw}"/>
   <parent link="carrier"/>
   <child link="linkage_point3_1"/>
-  <axis xyz="0.0 -0.0 -1.0"/>
+  <axis xyz="0.0 -0.0 1.0"/>
   <dynamics damping="${rotational_joint_damping}" friction="${rotational_joint_friction}"/>
   <limit effort="100" velocity="100"/>

Commit message: fix runge

File: urdf/cooperative_transportation_4ws.xacro (robot description, xacro)
@@ -43,6 +43,6 @@
 <xacro:property name="rotational_joint_friction" value="${rotational_joint_mu * gravitational_acceleration * carrier_inertia_coef/3}" />
 <!-- wheelの接地面の摩擦などを定義 -->
-<xacro:property name="wheel_surface_mu1" value="1.0"/>
-<xacro:property name="wheel_surface_mu2" value="0.8" />
+<xacro:property name="wheel_surface_mu1" value="0.8"/>
+<xacro:property name="wheel_surface_mu2" value="0.6" />
 <xacro:property name="wheel_kp" value="2e4" />
 <xacro:property name="wheel_kd" value="5.0" />

Commit message: 2025101718

File: urdf/cooperative_transportation_4ws.xacro (robot description, xacro)
@@ -20,5 +20,5 @@
 <xacro:property name="vehicle_inertia_coef" value="${sim_body_mass/fusion_vehicle_body_mass}" />
 <!-- 車輪 -->
-<xacro:property name="fusion_wheel_mass" value="${sim_wheel_mass}" />
+<xacro:property name="fusion_wheel_mass" value="20.0" />
 <xacro:property name="sim_wheel_mass" value="8.0" />
 <xacro:property name="wheel_inertia_coef" value="${sim_wheel_mass/fusion_wheel_mass}" />
@@ -31,19 +31,19 @@
 <xacro:property name="sliding_mechanism_mass" value="36.58325703660448" />
 <!-- 摺動機構 -->
-<xacro:property name="sliding_mechanism_damping" value="${(0.5*2*sqrt(100000*(carrier_inertia_coef/3 + linkage_point_mass)))/5.0}" /> <!-- ばね定数：1000~10000, 割合：50%-->
+<xacro:property name="sliding_mechanism_damping" value="${(0.5*2*sqrt(100000*(sim_carrier_mass/3 + linkage_point_mass)))/5.0}" /> <!-- ばね定数：1000~10000, 割合：50%-->
 <xacro:property name="sliding_mechanism_mu" value="0.3" />
-<xacro:property name="sliding_mechanism_friction" value="${sliding_mechanism_mu*gravitational_acceleration*(carrier_inertia_coef/3 + linkage_point_mass)}" />
+<xacro:property name="sliding_mechanism_friction" value="${sliding_mechanism_mu*gravitational_acceleration*(sim_carrier_mass/3 + linkage_point_mass)}" />
 <!-- ステアリング -->
-<xacro:property name="steering_damping" value="1.0" />
+<xacro:property name="steering_damping" value="5.0" />
 <xacro:property name="steering_mu" value="0.001" />
-<xacro:property name="steering_friction" value="${steering_mu * gravitational_acceleration * 0.25*(carrier_inertia_coef/3 + linkage_point_mass + sliding_mechanism_mass + sim_body_mass)}" />
+<xacro:property name="steering_friction" value="${steering_mu * gravitational_acceleration * 0.25*(sim_carrier_mass/3 + linkage_point_mass + sliding_mechanism_mass + sim_body_mass)}" />
 <!-- 摺動機構に乗っかている回転関節 -->
 <xacro:property name="rotational_joint_damping" value="0.02" />
 <xacro:property name="rotational_joint_mu" value="0.001" />
-<xacro:property name="rotational_joint_friction" value="${rotational_joint_mu * gravitational_acceleration * carrier_inertia_coef/3}" />
+<xacro:property name="rotational_joint_friction" value="${rotational_joint_mu * gravitational_acceleration * sim_carrier_mass/3}" />
 <!-- wheelの接地面の摩擦などを定義 -->
 <xacro:property name="wheel_surface_mu1" value="0.8"/>
 <xacro:property name="wheel_surface_mu2" value="0.6" />
-<xacro:property name="wheel_kp" value="2e4" />
+<xacro:property name="wheel_kp" value="2e7" />
 <xacro:property name="wheel_kd" value="5.0" />
 <xacro:property name="wheel_minDepth" value="0.01" />
@@ -1155,5 +1155,5 @@
   <dynamics damping="${wheel_joint_damping}" friction="${wheel_joint_friction}"/>
   <axis xyz="0.0 1.0 -0.0"/>
-  <limit effort="100.0" velocity="200.0"/>
+  <limit effort="100.0" velocity="${1.0/0.153}"/>
 </joint>
 <joint name="v1_rear_right_steering" type="revolute">
@@ -1210,5 +1210,5 @@
   <dynamics damping="${wheel_joint_damping}" friction="${wheel_joint_friction}"/>
   <axis xyz="0.0 1.0 -0.0"/>
-  <limit effort="100.0" velocity="200.0"/>
+  <limit effort="100.0" velocity="${1.0/0.153}"/>
 </joint>
 <joint name="v1_front_left_wheel_rotation" type="continuous">
@@ -1218,5 +1218,5 @@
   <dynamics damping="${wheel_joint_damping}" friction="${wheel_joint_friction}"/>
   <axis xyz="0.0 1.0 -0.0"/>
-  <limit effort="100.0" velocity="200.0"/>
+  <limit effort="100.0" velocity="${1.0/0.153}"/>
 </joint>
 <joint name="v1_rear_left_wheel_rotation" type="continuous">
@@ -1226,5 +1226,5 @@
   <dynamics damping="${wheel_joint_damping}" friction="${wheel_joint_friction}"/>
   <axis xyz="0.0 1.0 -0.0"/>
-  <limit effort="100.0" velocity="200.0"/>
+  <limit effort="100.0" velocity="${1.0/0.153}"/>
 </joint>
 <!-- <joint name="linkage1_rotation" type="continuous">
@@ -1326,5 +1326,5 @@
   <dynamics damping="${wheel_joint_damping}" friction="${wheel_joint_friction}"/>
   <axis xyz="0.0 1.0 -0.0"/>
-  <limit effort="100.0" velocity="200.0"/>
+  <limit effort="100.0" velocity="${1.0/0.153}"/>
 </joint>
 <joint name="v2_rear_right_wheel_rotation" type="continuous">
@@ -1334,5 +1334,5 @@
   <dynamics damping="${wheel_joint_damping}" friction="${wheel_joint_friction}"/>
   <axis xyz="-0.0 1.0 -0.0"/>
-  <limit effort="100.0" velocity="200.0"/>
+  <limit effort="100.0" velocity="${1.0/0.153}"/>
 </joint>
 <joint name="v2_front_left_wheel_rotation" type="continuous">
@@ -1342,5 +1342,5 @@
   <dynamics damping="${wheel_joint_damping}" friction="${wheel_joint_friction}"/>
   <axis xyz="0.0 1.0 -0.0"/>
-  <limit effort="100.0" velocity="200.0"/>
+  <limit effort="100.0" velocity="${1.0/0.153}"/>
 </joint>
 <joint name="v2_rear_left_wheel_rotation" type="continuous">
@@ -1350,5 +1350,5 @@
   <dynamics damping="${wheel_joint_damping}" friction="${wheel_joint_friction}"/>
   <axis xyz="-0.0 1.0 -0.0"/>
-  <limit effort="100.0" velocity="200.0"/>
+  <limit effort="100.0" velocity="${1.0/0.153}"/>
 </joint>
 <joint name="v3_sliding_machine_to_body" type="fixed">
@@ -1405,5 +1405,5 @@
   <dynamics damping="${wheel_joint_damping}" friction="${wheel_joint_friction}"/>
   <axis xyz="0.0 1.0 -0.0"/>
-  <limit effort="100.0" velocity="200.0"/>
+  <limit effort="100.0" velocity="${1.0/0.153}"/>
 </joint>
 <joint name="v3_rear_right_wheel_rotation" type="continuous">
@@ -1413,5 +1413,5 @@
   <dynamics damping="${wheel_joint_damping}" friction="${wheel_joint_friction}"/>
   <axis xyz="0.0 1.0 -0.0"/>
-  <limit effort="100.0" velocity="200.0"/>
+  <limit effort="100.0" velocity="${1.0/0.153}"/>
 </joint>
 <joint name="v3_front_left_wheel_rotation" type="continuous">
@@ -1421,5 +1421,5 @@
   <dynamics damping="${wheel_joint_damping}" friction="${wheel_joint_friction}"/>
   <axis xyz="0.0 1.0 -0.0"/>
-  <limit effort="100.0" velocity="200.0"/>
+  <limit effort="100.0" velocity="${1.0/0.153}"/>
 </joint>
 <joint name="v3_rear_left_wheel_rotation" type="continuous">
@@ -1429,5 +1429,5 @@
   <dynamics damping="${wheel_joint_damping}" friction="${wheel_joint_friction}"/>
   <axis xyz="0.0 1.0 -0.0"/>
-  <limit effort="100.0" velocity="200.0"/>
+  <limit effort="100.0" velocity="${1.0/0.153}"/>
 </joint>
 <joint name="linkage_point_to_v1" type="prismatic">

Commit message: y2

File: urdf/cooperative_transportation_4ws.xacro (robot description, xacro)
@@ -43,6 +43,6 @@
 <xacro:property name="rotational_joint_friction" value="${rotational_joint_mu * gravitational_acceleration * sim_carrier_mass/3}" />
 <!-- wheelの接地面の摩擦などを定義 -->
-<xacro:property name="wheel_surface_mu1" value="0.8"/>
-<xacro:property name="wheel_surface_mu2" value="0.6" />
+<xacro:property name="wheel_surface_mu1" value="0.7"/>
+<xacro:property name="wheel_surface_mu2" value="0.5" />
 <xacro:property name="wheel_kp" value="2e7" />
 <xacro:property name="wheel_kd" value="5.0" />
