Commit message: 20251114

File: urdf/cooperative_transportation_4ws_real.xacro (robot description, xacro)
@@ -57,27 +57,7 @@
 <xacro:include filename="$(find cooperative_transportation_4ws_description)/urdf/cooperative_transportation_4ws.gazebo" />
 <link name="base_link"/>
-<!-- <link name="carrier">
-  <inertial>
-    <origin xyz="0 0 0" rpy="0 0 0"/>
-    <mass value="2052.2363345901408"/>
-    <inertia ixx="586.219446" iyy="586.234405" izz="1171.807086" ixy="0.007184" iyz="0.0" ixz="0.0"/>
-  </inertial>
-  <visual>
-    <origin xyz="0 0 -0.6559999999999989" rpy="0 0 0"/>
-    <geometry>
-      <mesh filename="package://cooperative_transportation_4ws_description/meshes/base_link.stl" scale="0.001 0.001 0.001"/>
-    </geometry>
-    <material name="yellow"/>
-  </visual>
-  <collision>
-    <origin xyz="0 0 -0.6559999999999989" rpy="0 0 0"/>
-    <geometry>
-      <mesh filename="package://cooperative_transportation_4ws_description/meshes/base_link.stl" scale="0.001 0.001 0.001"/>
-    </geometry>
-  </collision>
-</link> -->
 <link name="carrier">
   <inertial>
-    <origin xyz="-0.00038139052519531075 0.05527097122796802 0.0" rpy="0 0 0"/>
+    <origin xyz="-0.00038139052519531075 0.0 0.0" rpy="0 0 0"/>
     <mass value="${sim_carrier_mass}"/>
     <inertia ixx="${carrier_inertia_coef*586.219446}" iyy="${carrier_inertia_coef*586.234405}" izz="${carrier_inertia_coef*1171.807086}" ixy="${carrier_inertia_coef*0.007184}" iyz="0.0" ixz="0.0"/>

Commit message: 20251118

File: urdf/cooperative_transportation_4ws_real.xacro (robot description, xacro)
@@ -28,5 +28,5 @@
 <xacro:property name="hinge_inertia_coef" value="${sim_hinge_mass/fusion_hinge_mass}" />
 <xacro:property name="wheel_joint_damping" value="  1.0" />
-<xacro:property name="wheel_joint_mu" value="0.1" />
+<xacro:property name="wheel_joint_mu" value="0.01" />
 <xacro:property name="wheel_joint_friction" value="${wheel_joint_mu* gravitational_acceleration * sim_wheel_mass }" />
 <xacro:property name="carrier_mass" value="2052.2363345901408" />
@@ -40,5 +40,5 @@
 <!-- ステアリング -->
 <xacro:property name="steering_damping" value="1.0" />
-<xacro:property name="steering_mu" value="0.01" />
+<xacro:property name="steering_mu" value="0.05" />
 <xacro:property name="steering_friction" value="${steering_mu * gravitational_acceleration * 0.25*(sim_carrier_mass/3 + linkage_point_mass + sliding_mechanism_mass + sim_body_mass)}" />
 <!-- 摺動機構に乗っかている回転関節 -->
@@ -47,5 +47,5 @@
 <xacro:property name="rotational_joint_friction" value="${rotational_joint_mu * gravitational_acceleration * sim_carrier_mass/3}" />
 <!-- wheelの接地面の摩擦などを定義 -->
-<xacro:property name="wheel_surface_mu1" value="0.7"/>
+<xacro:property name="wheel_surface_mu1" value="0.8"/>
 <xacro:property name="wheel_surface_mu2" value="0.5" />
 <xacro:property name="wheel_kp" value="2e7" />
@@ -93,5 +93,5 @@
     <origin xyz="0 0 0" rpy="1.57 0 0"/>
     <geometry>
-      <cylinder radius="0.153" length="0.07"/>
+      <cylinder radius="0.16" length="0.07"/>
     </geometry>
   </collision>
@@ -253,5 +253,5 @@
     <origin xyz="0 0 0" rpy="1.57 0 0"/>
     <geometry>
-      <cylinder radius="0.153" length="0.07"/>
+      <cylinder radius="0.16" length="0.07"/>
     </geometry>
     <surface>
@@ -295,5 +295,5 @@
     <origin xyz="0 0 0" rpy="1.57 0 0"/>
     <geometry>
-      <cylinder radius="0.153" length="0.07"/>
+      <cylinder radius="0.16" length="0.07"/>
     </geometry>
     <surface>
@@ -337,5 +337,5 @@
     <origin xyz="0 0 0" rpy="1.57 0 0"/>
     <geometry>
-      <cylinder radius="0.153" length="0.07"/>
+      <cylinder radius="0.16" length="0.07"/>
     </geometry>
     <surface>
@@ -579,5 +579,5 @@
     <origin xyz="0 0 0" rpy="1.57 0 0"/>
     <geometry>
-      <cylinder radius="0.153" length="0.07"/>
+      <cylinder radius="0.16" length="0.07"/>
     </geometry>
     <surface>
@@ -621,5 +621,5 @@
     <origin xyz="0 0 0" rpy="1.57 0 0"/>
     <geometry>
-      <cylinder radius="0.153" length="0.07"/>
+      <cylinder radius="0.16" length="0.07"/>
     </geometry>
     <surface>
@@ -663,5 +663,5 @@
     <origin xyz="0 0 0" rpy="1.57 0 0"/>
     <geometry>
-      <cylinder radius="0.153" length="0.07"/>
+      <cylinder radius="0.16" length="0.07"/>
     </geometry>
     <surface>
@@ -705,5 +705,5 @@
     <origin xyz="0 0 0" rpy="1.57 0 0"/>
     <geometry>
-      <cylinder radius="0.153" length="0.07"/>
+      <cylinder radius="0.16" length="0.07"/>
     </geometry>
     <surface>
@@ -887,5 +887,5 @@
     <origin xyz="0 0 0" rpy="1.57 0 0"/>
     <geometry>
-      <cylinder radius="0.153" length="0.07"/>
+      <cylinder radius="0.16" length="0.07"/>
     </geometry>
     <surface>
@@ -929,5 +929,5 @@
     <origin xyz="0 0 0" rpy="1.57 0 0"/>
     <geometry>
-      <cylinder radius="0.153" length="0.07"/>
+      <cylinder radius="0.16" length="0.07"/>
     </geometry>
     <surface>
@@ -971,5 +971,5 @@
     <origin xyz="0 0 0" rpy="1.57 0 0"/>
     <geometry>
-      <cylinder radius="0.153" length="0.07"/>
+      <cylinder radius="0.16" length="0.07"/>
     </geometry>
     <surface>
@@ -1013,5 +1013,5 @@
     <origin xyz="0 0 0" rpy="1.57 0 0"/>
     <geometry>
-      <cylinder radius="0.153" length="0.07"/>
+      <cylinder radius="0.16" length="0.07"/>
     </geometry>
     <surface>

Commit message: 20251124

File: urdf/cooperative_transportation_4ws_real.xacro (robot description, xacro)
@@ -40,5 +40,5 @@
 <!-- ステアリング -->
 <xacro:property name="steering_damping" value="1.0" />
-<xacro:property name="steering_mu" value="0.05" />
+<xacro:property name="steering_mu" value="0.02" />
 <xacro:property name="steering_friction" value="${steering_mu * gravitational_acceleration * 0.25*(sim_carrier_mass/3 + linkage_point_mass + sliding_mechanism_mass + sim_body_mass)}" />
 <!-- 摺動機構に乗っかている回転関節 -->
@@ -48,5 +48,5 @@
 <!-- wheelの接地面の摩擦などを定義 -->
 <xacro:property name="wheel_surface_mu1" value="0.8"/>
-<xacro:property name="wheel_surface_mu2" value="0.5" />
+<xacro:property name="wheel_surface_mu2" value="0.4" />
 <xacro:property name="wheel_kp" value="2e7" />
 <xacro:property name="wheel_kd" value="5.0" />

Commit message: fix sliding machine joint

File: urdf/cooperative_transportation_4ws_real.xacro (robot description, xacro)
@@ -1420,5 +1420,5 @@
   <child link="v1_sliding_machine_1"/>
   <dynamics damping="${sliding_mechanism_damping}" friction="${sliding_mechanism_friction}"/>
-  <axis xyz="0 -1 0"/>
+  <axis xyz="0 1 0"/>
   <limit upper="0.0" lower="0.0" effort="10" velocity="10"/>
 </joint>
@@ -1428,5 +1428,5 @@
   <child link="v2_sliding_machine_1"/>
   <dynamics damping="${sliding_mechanism_damping}" friction="${sliding_mechanism_friction}"/>
-  <axis xyz="0 -1 0"/>
+  <axis xyz="0 1 0"/>
   <limit upper="0.0" lower="0.0" effort="10" velocity="10"/>
 </joint>
@@ -1436,5 +1436,5 @@
   <child link="v3_sliding_machine_1"/>
   <dynamics damping="${sliding_mechanism_damping}" friction="${sliding_mechanism_friction}"/>
-  <axis xyz="0 -1 0"/>
+  <axis xyz="0 1 0"/>
   <limit upper="0.0" lower="0.0" effort="10" velocity="10"/>
 </joint>

Commit message: 2025120215

File: urdf/cooperative_transportation_4ws_real.xacro (robot description, xacro)
@@ -21,5 +21,5 @@
 <!-- 車輪 -->
 <xacro:property name="fusion_wheel_mass" value="20.0" />
-<xacro:property name="sim_wheel_mass" value="8.0" />
+<xacro:property name="sim_wheel_mass" value="15.0" />
 <xacro:property name="wheel_inertia_coef" value="${sim_wheel_mass/fusion_wheel_mass}" />
 <!-- hinge -->
@@ -93,5 +93,5 @@
     <origin xyz="0 0 0" rpy="1.57 0 0"/>
     <geometry>
-      <cylinder radius="0.16" length="0.07"/>
+      <cylinder radius="0.16" length="0.08"/>
     </geometry>
   </collision>
@@ -253,5 +253,5 @@
     <origin xyz="0 0 0" rpy="1.57 0 0"/>
     <geometry>
-      <cylinder radius="0.16" length="0.07"/>
+      <cylinder radius="0.16" length="0.08"/>
     </geometry>
     <surface>
@@ -295,5 +295,5 @@
     <origin xyz="0 0 0" rpy="1.57 0 0"/>
     <geometry>
-      <cylinder radius="0.16" length="0.07"/>
+      <cylinder radius="0.16" length="0.08"/>
     </geometry>
     <surface>
@@ -337,5 +337,5 @@
     <origin xyz="0 0 0" rpy="1.57 0 0"/>
     <geometry>
-      <cylinder radius="0.16" length="0.07"/>
+      <cylinder radius="0.16" length="0.08"/>
     </geometry>
     <surface>
@@ -579,5 +579,5 @@
     <origin xyz="0 0 0" rpy="1.57 0 0"/>
     <geometry>
-      <cylinder radius="0.16" length="0.07"/>
+      <cylinder radius="0.16" length="0.08"/>
     </geometry>
     <surface>
@@ -621,5 +621,5 @@
     <origin xyz="0 0 0" rpy="1.57 0 0"/>
     <geometry>
-      <cylinder radius="0.16" length="0.07"/>
+      <cylinder radius="0.16" length="0.08"/>
     </geometry>
     <surface>
@@ -663,5 +663,5 @@
     <origin xyz="0 0 0" rpy="1.57 0 0"/>
     <geometry>
-      <cylinder radius="0.16" length="0.07"/>
+      <cylinder radius="0.16" length="0.08"/>
     </geometry>
     <surface>
@@ -705,5 +705,5 @@
     <origin xyz="0 0 0" rpy="1.57 0 0"/>
     <geometry>
-      <cylinder radius="0.16" length="0.07"/>
+      <cylinder radius="0.16" length="0.08"/>
     </geometry>
     <surface>
@@ -887,5 +887,5 @@
     <origin xyz="0 0 0" rpy="1.57 0 0"/>
     <geometry>
-      <cylinder radius="0.16" length="0.07"/>
+      <cylinder radius="0.16" length="0.08"/>
     </geometry>
     <surface>
@@ -929,5 +929,5 @@
     <origin xyz="0 0 0" rpy="1.57 0 0"/>
     <geometry>
-      <cylinder radius="0.16" length="0.07"/>
+      <cylinder radius="0.16" length="0.08"/>
     </geometry>
     <surface>
@@ -971,5 +971,5 @@
     <origin xyz="0 0 0" rpy="1.57 0 0"/>
     <geometry>
-      <cylinder radius="0.16" length="0.07"/>
+      <cylinder radius="0.16" length="0.08"/>
     </geometry>
     <surface>
@@ -1013,5 +1013,5 @@
     <origin xyz="0 0 0" rpy="1.57 0 0"/>
     <geometry>
-      <cylinder radius="0.16" length="0.07"/>
+      <cylinder radius="0.16" length="0.08"/>
     </geometry>
     <surface>
