Commit message: Modify the non-holonomic constraints of the wheels

File: urdf/cooperative_transportation_4ws_real.xacro (robot description, xacro)
@@ -17,9 +17,9 @@
 <!-- 車両のbody-->
 <xacro:property name="fusion_vehicle_body_mass" value="2113.272311120373" />
-<xacro:property name="sim_body_mass" value="100" />
+<xacro:property name="sim_body_mass" value="70" />
 <xacro:property name="vehicle_inertia_coef" value="${sim_body_mass/fusion_vehicle_body_mass}" />
 <!-- 車輪 -->
 <xacro:property name="fusion_wheel_mass" value="20.0" />
-<xacro:property name="sim_wheel_mass" value="15.0" />
+<xacro:property name="sim_wheel_mass" value="8.0" />
 <xacro:property name="wheel_inertia_coef" value="${sim_wheel_mass/fusion_wheel_mass}" />
 <!-- hinge -->
@@ -27,6 +27,14 @@
 <xacro:property name="sim_hinge_mass" value="3.498237661363729" />
 <xacro:property name="hinge_inertia_coef" value="${sim_hinge_mass/fusion_hinge_mass}" />
+<!-- 荷台の連結点の棒 -->
+<xacro:property name="fusion_linkage_mass" value="16.301253040579397" />
+<xacro:property name="sim_linkage_mass" value="1.0" />
+<xacro:property name="linkage_inertia_coef" value="${sim_linkage_mass/fusion_linkage_mass}" />
+<!-- 車軸の棒 -->
+<xacro:property name="fusion_axle_mass" value="12.646385127140846" />
+<xacro:property name="sim_axle_mass" value="1.0" />
+<xacro:property name="axle_inertia_coef" value="${sim_axle_mass/fusion_axle_mass}" />
 <xacro:property name="wheel_joint_damping" value="  1.0" />
-<xacro:property name="wheel_joint_mu" value="0.01" />
+<xacro:property name="wheel_joint_mu" value="0.001" />
 <xacro:property name="wheel_joint_friction" value="${wheel_joint_mu* gravitational_acceleration * sim_wheel_mass }" />
 <xacro:property name="carrier_mass" value="2052.2363345901408" />
@@ -35,10 +43,10 @@
 <xacro:property name="sliding_mechanism_mass" value="36.58325703660448" />
 <!-- 摺動機構 -->
-<xacro:property name="sliding_mechanism_damping" value="${(0.5*2*sqrt(100000*(sim_carrier_mass/3 + linkage_point_mass)))/5.0}" /> <!-- ばね定数：1000~10000, 割合：50%-->
+<xacro:property name="sliding_mechanism_damping" value="10.0" /> <!-- ばね定数：1000~10000, 割合：50%-->
 <xacro:property name="sliding_mechanism_mu" value="0.3" />
 <xacro:property name="sliding_mechanism_friction" value="${sliding_mechanism_mu*gravitational_acceleration*(sim_carrier_mass/3 + linkage_point_mass)}" />
 <!-- ステアリング -->
-<xacro:property name="steering_damping" value="1.0" />
-<xacro:property name="steering_mu" value="0.02" />
+<xacro:property name="steering_damping" value="0.0" />
+<xacro:property name="steering_mu" value="0.06" />
 <xacro:property name="steering_friction" value="${steering_mu * gravitational_acceleration * 0.25*(sim_carrier_mass/3 + linkage_point_mass + sliding_mechanism_mass + sim_body_mass)}" />
 <!-- 摺動機構に乗っかている回転関節 -->
@@ -48,9 +56,9 @@
 <!-- wheelの接地面の摩擦などを定義 -->
 <xacro:property name="wheel_surface_mu1" value="0.8"/>
-<xacro:property name="wheel_surface_mu2" value="0.4" />
-<xacro:property name="wheel_kp" value="2e7" />
-<xacro:property name="wheel_kd" value="5.0" />
-<xacro:property name="wheel_minDepth" value="0.01" />
-<xacro:property name="wheel_maxVel" value="0.5" />
+<xacro:property name="wheel_surface_mu2" value="0.5" />
+<xacro:property name="wheel_kp" value="5e5" />
+<xacro:property name="wheel_kd" value="100.0" />
+<xacro:property name="wheel_minDepth" value="0.002" />
+<xacro:property name="wheel_maxVel" value="1.0" />
 <xacro:include filename="$(find cooperative_transportation_4ws_description)/urdf/materials.xacro" />
 <xacro:include filename="$(find cooperative_transportation_4ws_description)/urdf/cooperative_transportation_4ws.trans" />
@@ -93,5 +101,5 @@
     <origin xyz="0 0 0" rpy="1.57 0 0"/>
     <geometry>
-      <cylinder radius="0.16" length="0.08"/>
+      <cylinder radius="0.16" length="0.06"/>
     </geometry>
   </collision>
@@ -181,5 +189,5 @@
     <origin xyz="0.0009614087301266228 -8.103821973019787e-06 -0.13737493498310355" rpy="0 0 0"/>
     <mass value="${sim_body_mass}"/>
-    <inertia ixx="${vehicle_inertia_coef*114.688091}" iyy="${vehicle_inertia_coef*336.418835}" izz="${vehicle_inertia_coef*418.647558}" ixy="${vehicle_inertia_coef*0.010139}" iyz="${vehicle_inertia_coef*0.002956}" ixz="${vehicle_inertia_coef*-0.33997}"/>
+    <inertia ixx="${vehicle_inertia_coef*114.688091}" iyy="${vehicle_inertia_coef*336.418835}" izz="${vehicle_inertia_coef*418.647558}" ixy="${vehicle_inertia_coef*0.010139}" iyz="${vehicle_inertia_coef*0.002956}" ixz="${-vehicle_inertia_coef*0.33997}"/>
   </inertial>
   <visual>
@@ -200,6 +208,6 @@
   <inertial>
     <origin xyz="2.5142643989006785e-07 2.5406923826604144e-07 -0.014912246259013051" rpy="0 0 0"/>
-    <mass value="12.646385127140846"/>
-    <inertia ixx="0.752015" iyy="0.005192" izz="0.755318" ixy="0.0" iyz="0.0" ixz="0.0"/>
+    <mass value="${sim_axle_mass}"/>
+    <inertia ixx="${axle_inertia_coef*0.752015}" iyy="${axle_inertia_coef*0.005192}" izz="${axle_inertia_coef*0.755318}" ixy="0.0" iyz="0.0" ixz="0.0"/>
   </inertial>
   <visual>
@@ -220,6 +228,6 @@
   <inertial>
     <origin xyz="2.514264378916664e-07 2.5406916610154484e-07 -0.014912246259013162" rpy="0 0 0"/>
-    <mass value="12.64638512714101"/>
-    <inertia ixx="0.752015" iyy="0.005192" izz="0.755318" ixy="-0.0" iyz="0.0" ixz="-0.0"/>
+    <mass value="${sim_axle_mass}"/>
+    <inertia ixx="${axle_inertia_coef*0.752015}" iyy="${axle_inertia_coef*0.005192}" izz="${axle_inertia_coef*0.755318}" ixy="0.0" iyz="0.0" ixz="0.0"/>
   </inertial>
   <visual>
@@ -253,5 +261,5 @@
     <origin xyz="0 0 0" rpy="1.57 0 0"/>
     <geometry>
-      <cylinder radius="0.16" length="0.08"/>
+      <cylinder radius="0.16" length="0.06"/>
     </geometry>
     <surface>
@@ -265,5 +273,5 @@
           <!-- 強すぎるスティッキングを避けるためのスリップ（力依存） -->
           <slip1>0.001</slip1>   <!-- rolling -->
-          <slip2>0.0</slip2>     <!-- lateral（基本0でOK、必要なら微小） -->
+          <slip2>0.03</slip2>     <!-- lateral（基本0でOK、必要なら微小） -->
         </ode>
       </friction>
@@ -295,5 +303,5 @@
     <origin xyz="0 0 0" rpy="1.57 0 0"/>
     <geometry>
-      <cylinder radius="0.16" length="0.08"/>
+      <cylinder radius="0.16" length="0.06"/>
     </geometry>
     <surface>
@@ -307,5 +315,5 @@
           <!-- 強すぎるスティッキングを避けるためのスリップ（力依存） -->
           <slip1>0.001</slip1>   <!-- rolling -->
-          <slip2>0.0</slip2>     <!-- lateral（基本0でOK、必要なら微小） -->
+          <slip2>0.03</slip2>     <!-- lateral（基本0でOK、必要なら微小） -->
         </ode>
       </friction>
@@ -337,5 +345,5 @@
     <origin xyz="0 0 0" rpy="1.57 0 0"/>
     <geometry>
-      <cylinder radius="0.16" length="0.08"/>
+      <cylinder radius="0.16" length="0.06"/>
     </geometry>
     <surface>
@@ -349,5 +357,5 @@
           <!-- 強すぎるスティッキングを避けるためのスリップ（力依存） -->
           <slip1>0.001</slip1>   <!-- rolling -->
-          <slip2>0.0</slip2>     <!-- lateral（基本0でOK、必要なら微小） -->
+          <slip2>0.03</slip2>     <!-- lateral（基本0でOK、必要なら微小） -->
         </ode>
       </friction>
@@ -366,6 +374,6 @@
   <inertial>
     <origin xyz="2.514264050290649e-07 7.029564128707699e-08 -0.11791981845688482" rpy="0 0 0"/>
-    <mass value="16.301253040579397"/>
-    <inertia ixx="0.104905" iyy="0.104905" izz="0.020865" ixy="0.0" iyz="0.0" ixz="0.0"/>
+    <mass value="1.0"/>
+    <inertia ixx="${linkage_inertia_coef*0.104905}" iyy="${linkage_inertia_coef*0.104905}" izz="${linkage_inertia_coef*0.020865}" ixy="0.0" iyz="0.0" ixz="0.0"/>
   </inertial>
   <visual>
@@ -386,6 +394,6 @@
   <inertial>
     <origin xyz="3.2372278280234923e-07 -1.568761989201306e-07 -0.11791981845688582" rpy="0 0 0"/>
-    <mass value="16.30125304057939"/>
-    <inertia ixx="0.104905" iyy="0.104905" izz="0.020865" ixy="0.0" iyz="0.0" ixz="0.0"/>
+    <mass value="1.0"/>
+    <inertia ixx="${linkage_inertia_coef*0.104905}" iyy="${linkage_inertia_coef*0.104905}" izz="${linkage_inertia_coef*0.020865}" ixy="0.0" iyz="0.0" ixz="0.0"/>
   </inertial>
   <visual>
@@ -406,6 +414,6 @@
   <inertial>
     <origin xyz="-2.1871393585115584e-14 -1.837735197351975e-07 -0.11791981845688337" rpy="0 0 0"/>
-    <mass value="16.301253040579386"/>
-    <inertia ixx="0.104905" iyy="0.104905" izz="0.020865" ixy="0.0" iyz="0.0" ixz="0.0"/>
+    <mass value="1.0"/>
+    <inertia ixx="${linkage_inertia_coef*0.104905}" iyy="${linkage_inertia_coef*0.104905}" izz="${linkage_inertia_coef*0.020865}" ixy="0.0" iyz="0.0" ixz="0.0"/>
   </inertial>
   <visual>
@@ -446,6 +454,6 @@
   <inertial>
     <origin xyz="3.2372281477677234e-07 2.689739853067863e-08 -0.014912246259013773" rpy="0 0 0"/>
-    <mass value="12.646385127140846"/>
-    <inertia ixx="0.752015" iyy="0.005192" izz="0.755318" ixy="0.0" iyz="0.0" ixz="0.0"/>
+    <mass value="${sim_axle_mass}"/>
+    <inertia ixx="${axle_inertia_coef*0.752015}" iyy="${axle_inertia_coef*0.005192}" izz="${axle_inertia_coef*0.755318}" ixy="0.0" iyz="0.0" ixz="0.0"/>
   </inertial>
   <visual>
@@ -466,6 +474,6 @@
   <inertial>
     <origin xyz="3.237228147212612e-07 2.6897325255959004e-08 -0.014912246259013828" rpy="0 0 0"/>
-    <mass value="12.64638512714101"/>
-    <inertia ixx="0.752015" iyy="0.005192" izz="0.755318" ixy="-0.0" iyz="0.0" ixz="-0.0"/>
+    <mass value="${sim_axle_mass}"/>
+    <inertia ixx="${axle_inertia_coef*0.752015}" iyy="${axle_inertia_coef*0.005192}" izz="${axle_inertia_coef*0.755318}" ixy="0.0" iyz="0.0" ixz="0.0"/>
   </inertial>
   <visual>
@@ -579,5 +587,5 @@
     <origin xyz="0 0 0" rpy="1.57 0 0"/>
     <geometry>
-      <cylinder radius="0.16" length="0.08"/>
+      <cylinder radius="0.16" length="0.06"/>
     </geometry>
     <surface>
@@ -591,5 +599,5 @@
           <!-- 強すぎるスティッキングを避けるためのスリップ（力依存） -->
           <slip1>0.001</slip1>   <!-- rolling -->
-          <slip2>0.0</slip2>     <!-- lateral（基本0でOK、必要なら微小） -->
+          <slip2>0.03</slip2>     <!-- lateral（基本0でOK、必要なら微小） -->
         </ode>
       </friction>
@@ -621,5 +629,5 @@
     <origin xyz="0 0 0" rpy="1.57 0 0"/>
     <geometry>
-      <cylinder radius="0.16" length="0.08"/>
+      <cylinder radius="0.16" length="0.06"/>
     </geometry>
     <surface>
@@ -633,5 +641,5 @@
           <!-- 強すぎるスティッキングを避けるためのスリップ（力依存） -->
           <slip1>0.001</slip1>   <!-- rolling -->
-          <slip2>0.0</slip2>     <!-- lateral（基本0でOK、必要なら微小） -->
+          <slip2>0.03</slip2>     <!-- lateral（基本0でOK、必要なら微小） -->
         </ode>
       </friction>
@@ -663,5 +671,5 @@
     <origin xyz="0 0 0" rpy="1.57 0 0"/>
     <geometry>
-      <cylinder radius="0.16" length="0.08"/>
+      <cylinder radius="0.16" length="0.06"/>
     </geometry>
     <surface>
@@ -675,5 +683,5 @@
           <!-- 強すぎるスティッキングを避けるためのスリップ（力依存） -->
           <slip1>0.001</slip1>   <!-- rolling -->
-          <slip2>0.0</slip2>     <!-- lateral（基本0でOK、必要なら微小） -->
+          <slip2>0.03</slip2>     <!-- lateral（基本0でOK、必要なら微小） -->
         </ode>
       </friction>
@@ -705,5 +713,5 @@
     <origin xyz="0 0 0" rpy="1.57 0 0"/>
     <geometry>
-      <cylinder radius="0.16" length="0.08"/>
+      <cylinder radius="0.16" length="0.06"/>
     </geometry>
     <surface>
@@ -717,5 +725,5 @@
           <!-- 強すぎるスティッキングを避けるためのスリップ（力依存） -->
           <slip1>0.001</slip1>   <!-- rolling -->
-          <slip2>0.0</slip2>     <!-- lateral（基本0でOK、必要なら微小） -->
+          <slip2>0.03</slip2>     <!-- lateral（基本0でOK、必要なら微小） -->
         </ode>
       </friction>
@@ -754,6 +762,6 @@
   <inertial>
     <origin xyz="1.0880185641326534e-14 7.682743330406083e-14 -0.014912246259012052" rpy="0 0 0"/>
-    <mass value="12.646385127140846"/>
-    <inertia ixx="0.752015" iyy="0.005192" izz="0.755318" ixy="0.0" iyz="0.0" ixz="0.0"/>
+    <mass value="${sim_axle_mass}"/>
+    <inertia ixx="${axle_inertia_coef*0.752015}" iyy="${axle_inertia_coef*0.005192}" izz="${axle_inertia_coef*0.755318}" ixy="0.0" iyz="0.0" ixz="0.0"/>
   </inertial>
   <visual>
@@ -774,6 +782,6 @@
   <inertial>
     <origin xyz="9.658940314238862e-15 4.6629367034256575e-15 -0.014912246259011386" rpy="0 0 0"/>
-    <mass value="12.64638512714101"/>
-    <inertia ixx="0.752015" iyy="0.005192" izz="0.755318" ixy="-0.0" iyz="0.0" ixz="-0.0"/>
+    <mass value="${sim_axle_mass}"/>
+    <inertia ixx="${axle_inertia_coef*0.752015}" iyy="${axle_inertia_coef*0.005192}" izz="${axle_inertia_coef*0.755318}" ixy="0.0" iyz="0.0" ixz="0.0"/>
   </inertial>
   <visual>
@@ -887,5 +895,5 @@
     <origin xyz="0 0 0" rpy="1.57 0 0"/>
     <geometry>
-      <cylinder radius="0.16" length="0.08"/>
+      <cylinder radius="0.16" length="0.06"/>
     </geometry>
     <surface>
@@ -899,5 +907,5 @@
           <!-- 強すぎるスティッキングを避けるためのスリップ（力依存） -->
           <slip1>0.001</slip1>   <!-- rolling -->
-          <slip2>0.0</slip2>     <!-- lateral（基本0でOK、必要なら微小） -->
+          <slip2>0.03</slip2>     <!-- lateral（基本0でOK、必要なら微小） -->
         </ode>
       </friction>
@@ -929,5 +937,5 @@
     <origin xyz="0 0 0" rpy="1.57 0 0"/>
     <geometry>
-      <cylinder radius="0.16" length="0.08"/>
+      <cylinder radius="0.16" length="0.06"/>
     </geometry>
     <surface>
@@ -941,5 +949,5 @@
           <!-- 強すぎるスティッキングを避けるためのスリップ（力依存） -->
           <slip1>0.001</slip1>   <!-- rolling -->
-          <slip2>0.0</slip2>     <!-- lateral（基本0でOK、必要なら微小） -->
+          <slip2>0.03</slip2>     <!-- lateral（基本0でOK、必要なら微小） -->
         </ode>
       </friction>
@@ -971,5 +979,5 @@
     <origin xyz="0 0 0" rpy="1.57 0 0"/>
     <geometry>
-      <cylinder radius="0.16" length="0.08"/>
+      <cylinder radius="0.16" length="0.06"/>
     </geometry>
     <surface>
@@ -983,5 +991,5 @@
           <!-- 強すぎるスティッキングを避けるためのスリップ（力依存） -->
           <slip1>0.001</slip1>   <!-- rolling -->
-          <slip2>0.0</slip2>     <!-- lateral（基本0でOK、必要なら微小） -->
+          <slip2>0.03</slip2>     <!-- lateral（基本0でOK、必要なら微小） -->
         </ode>
       </friction>
@@ -1013,5 +1021,5 @@
     <origin xyz="0 0 0" rpy="1.57 0 0"/>
     <geometry>
-      <cylinder radius="0.16" length="0.08"/>
+      <cylinder radius="0.16" length="0.06"/>
     </geometry>
     <surface>
@@ -1025,5 +1033,5 @@
           <!-- 強すぎるスティッキングを避けるためのスリップ（力依存） -->
           <slip1>0.001</slip1>   <!-- rolling -->
-          <slip2>0.0</slip2>     <!-- lateral（基本0でOK、必要なら微小） -->
+          <slip2>0.03</slip2>     <!-- lateral（基本0でOK、必要なら微小） -->
         </ode>
       </friction>
